Commit message: ..

File: model/starling2max.urdf (robot description, URDF)
Before this commit: robot starling2max, 5 links, 4 joints
Joints:
- joint prop0_joint: type None -> fixed
- joint prop1_joint: type None -> fixed
- joint prop2_joint: type None -> fixed
- joint prop3_joint: type None -> fixed

Commit message: . .

File: model/starling2max.urdf (robot description, URDF)
Before this commit: robot starling2max, 5 links, 4 joints
Links:
- link prop0_link: geometry visual mesh filename=./Starling2Max7040Prop.obj scale=0.001 0.001 0.001
- link prop1_link: geometry visual mesh filename=./Starling2Max7040Prop.obj scale=0.001 0.001 0.001
- link prop2_link: geometry visual mesh filename=./Starling2Max7040Prop.obj scale=0.001 0.001 0.001
- link prop3_link: geometry visual mesh filename=./Starling2Max7040Prop.obj scale=0.001 0.001 0.001
Joints:
- joint prop0_joint: type fixed -> None
- joint prop1_joint: type fixed -> None
- joint prop2_joint: type fixed -> None
- joint prop3_joint: type fixed -> None

Commit message: ..

File: model/starling2max.urdf (robot description, URDF)
Before this commit: robot starling2max, 5 links, 4 joints
Joints:
- joint prop0_joint: axis (none) -> 0 0 1; type fixed -> continuous
- joint prop1_joint: axis (none) -> 0 0 1; type fixed -> continuous
- joint prop2_joint: axis (none) -> 0 0 1; type fixed -> continuous
- joint prop3_joint: axis (none) -> 0 0 1; type fixed -> continuous

Commit message: ..

File: model/starling2max.urdf (robot description, URDF)
Before this commit: robot starling2max, 5 links, 4 joints
Joints:
- joint prop0_joint: axis 0 0 1 -> (none); type continuous -> fixed
- joint prop1_joint: axis 0 0 1 -> (none); type continuous -> fixed
- joint prop2_joint: axis 0 0 1 -> (none); type continuous -> fixed
- joint prop3_joint: axis 0 0 1 -> (none); type continuous -> fixed

Commit message: attach links on drone

File: model/starling2max.urdf (robot description, URDF)
Before this commit: robot starling2max, 5 links, 4 joints
Links:
- added link attach0_link
- added link attach1_link
- added link attach2_link
Joints:
- added joint attach0_joint: type fixed, parent base_link, child attach0_link, origin xyz=0.0 0.028867513459 -0.02 rpy=0.0 0.0 0.0
- added joint attach1_joint: type fixed, parent base_link, child attach1_link, origin xyz=-0.025 -0.01443375673 -0.02 rpy=0.0 0.0 0.0
- added joint attach2_joint: type fixed, parent base_link, child attach2_link, origin xyz=0.025 -0.01443375673 -0.02 rpy=0.0 0.0 0.0

Commit message: triangle

File: model/starling2max.urdf (robot description, URDF)
Before this commit: robot starling2max, 8 links, 7 joints
Joints:
- joint attach0_joint: origin xyz=0.0 0.028867513459 -0.02 rpy=0.0 0.0 0.0 -> xyz=0.028867513459 0.0 -0.02 rpy=0.0 0.0 0.0
- joint attach1_joint: origin xyz=-0.025 -0.01443375673 -0.02 rpy=0.0 0.0 0.0 -> xyz=-0.01443375673 0.025 -0.02 rpy=0.0 0.0 0.0
- joint attach2_joint: origin xyz=0.025 -0.01443375673 -0.02 rpy=0.0 0.0 0.0 -> xyz=-0.01443375673 -0.025 -0.02 rpy=0.0 0.0 0.0
